File: USB2514B.kicad_sch (KiCad schematic)
At the start: 40 parts, among them J1 USB_A, J2 USB_C_Receptacle_USB2.0_16P, J3 USB_A, J4 USB_A, J6 USB_A, U1 USB2514B_Bi, U10 USBLC6-2P6, U11 USBLC6-2P6, U2 USBLC6-2P6, U4 MCP1703Ax-330xxTT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

Commit message: Added board outline via Edge.Cuts traces
Parts:
- added H1, H2, H3, H4: MountingHole, MountingHole:MountingHole_2.2mm_M2, symbol Mechanical:MountingHole
Other:
- note added: "Mounting Holes"
- moved on the sheet: R6
