File: power_switch.kicad_sch (KiCad schematic)
At the start: 9 parts, among them U3 AP22615AWU

Commit message: Generate GBR files and add symbols information for JLC-PCB PCBA purchase
Parts:
- C13: LCSC Part # (none) -> C711098
- C16: LCSC Part # (none) -> C7200356
- C17: LCSC Part # (none) -> C3841584
- C27, C31: LCSC Part # (none) -> C126625
- FB2: LCSC Part # (none) -> C14709
- R10: LCSC Part # (none) -> C5634705
- R9: Distributo Link 2 https://www.digikey.fr/fr/products/detail/yageo/RT0402WRD07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 -> (none); Distributor Link 2 (none) -> https://www.digikey.fr/fr/products/detail/yageo/RT0402WRD07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; LCSC Part # (none) -> C25531
- U3: Distributor Link 1 (none) -> https://www.mouser.fr/fr/ProductDetail/Diodes-Incorporated/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; LCSC Part # (none) -> C2680357; Manufacturer (none) -> Diodes Incorporated; Manufacturer Part Number (none) -> AP22615AWU-7
Changed lines of the file:
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@@
+			)
+		)
+		(property "LCSC Part #" "C126625"
+			(at 193.04 82.55 0)
+			(effects
+				(font
+					(size 1.27 1.27)
+				)
+				(hide yes)
 			)
 		)
@@
 			)
 		)
+		(property "LCSC Part #" "C7200356"
+			(at 166.37 81.28 0)
+			(effects
+				(font
+					(size 1.27 1.27)
+				)
+				(hide yes)
+			)
+		)
 		(pin "1"
 		)
@@
 			)
 		)
-		(property "Distributo Link 2" "https://www.digikey.fr/fr/products/detail/yageo/RT0402WRD0710KL/5926796?s=N4IgTCBcDaIAQCUAqAGALCsB1BARFA7AIwoDSAMnCALoC%2BQA"
+		(property "Distributor Link 2" "https://www.digikey.fr/fr/products/detail/yageo/RT0402WRD0710KL/5926796?s=N4IgTCBcDaIAQCUAqAGALCsB1BARFA7AIwoDSAMnCALoC%2BQA"
+			(at 93.98 82.55 0)
+			(effects
+				(font
+					(size 1.27 1.27)
+				)
+				(hide yes)
+			)
+		)
+		(property "LCSC Part #" "C25531"
 			(at 93.98 82.55 0)
 			(effects
@@
 			)
 		)
+		(property "LCSC Part #" "C3841584"
+			(at 179.07 81.28 0)
+			(effects
+				(font
+					(size 1.27 1.27)
+				)
+				(hide yes)
+			)
+		)
 		(pin "1"
 		)
@@
 			)
 		)
+		(property "LCSC Part #" "C5634705"
+			(at 157.48 88.9 0)
+			(effects
+				(font
+					(size 1.27 1.27)
+				)
+				(hide yes)
+			)
+		)
 		(pin "1"
 		)
@@
 			)
 		)
+		(property "LCSC Part #" "C711098"
+			(at 104.14 81.28 0)
+			(effects
+				(font
+					(size 1.27 1.27)
+				)
+				(hide yes)
+			)
+		)
 		(pin "1"
 		)
@@
 			)
 		)
+		(property "Manufacturer" "Diodes Incorporated "
+			(at 144.78 80.01 0)
+			(effects
+				(font
+					(size 1.27 1.27)
+				)
+				(hide yes)
+			)
+		)
+		(property "Manufacturer Part Number" "AP22615AWU-7 "
+			(at 144.78 80.01 0)
+			(effects
+				(font
+					(size 1.27 1.27)
+				)
+				(hide yes)
+			)
+		)
+		(property "Distributor Link 1" "https://www.mouser.fr/fr/ProductDetail/Diodes-Incorporated/AP22615AWU-7?qs=lc2O%252BfHJPVZPFwwoXj6nyg%3D%3D"
+			(at 144.78 80.01 0)
+			(effects
+				(font
+					(size 1.27 1.27)
+				)
+				(hide yes)
+			)
+		)
+		(property "LCSC Part #" "C2680357"
+			(at 144.78 80.01 0)
+			(effects
+				(font
+					(size 1.27 1.27)
+				)
+				(hide yes)
+			)
+		)
 		(pin "6"
 		)
@@
 			)
 		)
+		(property "LCSC Part #" "C126625"
+			(at 204.47 82.55 0)
+			(effects
+				(font
+					(size 1.27 1.27)
+				)
+				(hide yes)
+			)
+		)
 		(pin "1"
 		)
@@
 			(at 198.12 77.47 90)
 			(effects
+				(font
+					(size 1.27 1.27)
+				)
+				(hide yes)
+			)
+		)
+		(property "LCSC Part #" "C14709"
+			(at 198.12 77.47 90)
+			(effects
